File: tklx/tklx.kicad_pcb (KiCad board)
At the start: 2 copper layers, 190 parts

Commit message: finished keyswitch layout
Parts:
- removed D72, D89: SOD-123, Diode_SMD:D_SOD-123
- removed MX72, MX89: MX-NoLED, MX_Only:MXOnly-1U-NoLED
- added D100: SOD-123, Diode_SMD:D_SOD-123, B.Cu at (47.6, 138.1)
- added D96: SOD-123, Diode_SMD:D_SOD-123, B.Cu at (47.6, 61.9)
- added D97: SOD-123, Diode_SMD:D_SOD-123, B.Cu at (47.6, 81.0)
- added D98: SOD-123, Diode_SMD:D_SOD-123, B.Cu at (47.6, 100.0)
- added D99: SOD-123, Diode_SMD:D_SOD-123, B.Cu at (47.6, 119.1)
- added MX100: MX-NoLED, MX_Only:MXOnly-1U-NoLED, F.Cu at (38.1, 133.3)
- added MX96: MX-NoLED, MX_Only:MXOnly-1U-NoLED, F.Cu at (38.1, 57.1)
- added MX97: MX-NoLED, MX_Only:MXOnly-1U-NoLED, F.Cu at (38.1, 76.2)
- added MX98: MX-NoLED, MX_Only:MXOnly-1U-NoLED, F.Cu at (38.1, 95.2)
- added MX99: MX-NoLED, MX_Only:MXOnly-1U-NoLED, F.Cu at (38.1, 114.3)
- D1, D10, D11, D12, D13, D14, D15, D16, D17, D18, D19, D2, D20, D21, D22, D23, D24, D25, D26, D27, D28, D29, D3, D30, D31, D32, D33, D34, D35, D36, D37, D38, D39, D4, D40, D41, D42, D43, D44, D45, D46, D47, D48, D49, D5, D50, D51, D52, D53, D54, D55, D56, D57, D58, D59, D6, D60, D61, D62, D63, D64, D65, D66, D67, D68, D69, D7, D70, D71, D73, D74, D75, D76, D77, D78, D79, D8, D80, D81, D82, D83, D84, D85, D86, D87, D88, D9, D90, D91, D92, D93, D94, D95: moved to B.Cu
- MX95: footprint MX_Only:MXOnly-1U-NoLED -> MX_Only:MXOnly-2U-NoLED
- moved MX91 332.0 mm to (412.0, 33.3)
- moved MX92 330.2 mm to (412.0, 57.1)
- moved MX94 329.5 mm to (412.0, 133.3)
- moved MX93 329.4 mm to (412.0, 76.2)
- moved MX90 315.5 mm to (392.9, 133.3)
- moved MX88 315.4 mm to (392.9, 114.3)
- moved MX81 314.9 mm to (373.9, 33.3)
- moved MX82 311.3 mm to (373.9, 57.1)
- moved MX87 311.1 mm to (392.9, 76.2)
- moved MX86 310.3 mm to (392.9, 57.1)
- moved MX84 309.7 mm to (373.9, 133.3)
- moved MX83 309.3 mm to (373.9, 76.2)
- moved D94 306.5 mm to (421.5, 138.1), turned to 90 degrees
- moved MX85 300.4 mm to (392.9, 33.3)
- moved D93 295.8 mm to (421.5, 81.0), turned to 90 degrees
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Connections:
- net COL10 renamed Net-(MX56-COL)
- net COL11 renamed Net-(MX62-COL)
- net COL15 renamed Net-(MX81-COL)
- net COL16 renamed Net-(MX85-COL)
- net COL17 renamed Net-(MX91-COL)
- net COL2 renamed Net-(MX12-COL)
- net COL3 renamed Net-(MX18-COL)
- net COL4 renamed Net-(MX24-COL)
- net COL5 renamed Net-(MX29-COL)
- net COL6 renamed Net-(MX34-COL)
- net COL7 renamed Net-(MX40-COL)
- net COL8 renamed Net-(MX45-COL)
- net COL9 renamed Net-(MX50-COL)
- D77 pad 1: ROW3 -> ROW4
- D79 pad 1: ROW1 -> ROW2
- D80 pad 1: ROW2 -> ROW3
- D84 pad 1: ROW4 -> ROW5
- D88 pad 1: ROW3 -> ROW4
- D94 pad 1: ROW4 -> ROW5
- D95 pad 1: ROW3 -> ROW1
- D95 pad 2: Net-(D9-A) -> Net-(D95-A)
- MX1 pad 1: COL0 -> COl1
- MX10 pad 1: COl1 -> Net-(MX10-COL)
- MX11 pad 1: COl1 -> Net-(MX10-COL)
- MX2 pad 1: COL0 -> COl1
- MX3 pad 1: COL0 -> COl1
- MX4 pad 1: COL0 -> COl1
- MX5 pad 1: COL0 -> COl1
- MX6 pad 1: COl1 -> Net-(MX10-COL)
- MX68 pad 1: COL12 -> Net-(MX68-COL)
- MX69 pad 1: COL12 -> Net-(MX68-COL)
- MX7 pad 1: COl1 -> Net-(MX10-COL)
- MX70 pad 1: COL12 -> Net-(MX68-COL)
- MX71 pad 1: COL12 -> Net-(MX68-COL)
- MX73 pad 1: COL12 -> Net-(MX73-COL)
- MX74 pad 1: COL13 -> Net-(MX73-COL)
- MX75 pad 1: COL13 -> Net-(MX73-COL)
- MX76 pad 1: COL13 -> Net-(MX73-COL)
- MX77 pad 1: COL13 -> Net-(MX73-COL)
- MX78 pad 1: COL14 -> Net-(MX78-COL)
- MX79 pad 1: COL14 -> Net-(MX78-COL)
- MX8 pad 1: COl1 -> Net-(MX10-COL)
- MX80 pad 1: COL14 -> Net-(MX78-COL)
- MX9 pad 1: COl1 -> Net-(MX10-COL)
- MX95 pad 1: COl1 -> Net-(MX78-COL)
- MX95 pad 2: Net-(D9-A) -> Net-(D95-A)

Commit message: finished microcontroller layout
Parts:
- moved D2 115.7 mm to (135.5, 173.8)
- moved D96 115.7 mm to (116.7, 154.8)
- moved D97 115.7 mm to (116.7, 173.8)
- moved D99 115.7 mm to (116.7, 211.9)
- moved MX1 115.7 mm to (126.2, 150.0)
- moved MX100 115.7 mm to (107.2, 226.2)
- moved MX3 115.7 mm to (126.2, 188.1)
- moved MX5 115.7 mm to (126.2, 226.2)
- moved MX96 115.7 mm to (107.2, 150.0)
- moved MX98 115.7 mm to (107.2, 188.1)
- moved D1 115.7 mm to (135.7, 154.8)
- moved D3 115.7 mm to (135.7, 192.9)
- moved D4 115.7 mm to (135.7, 211.9)
- moved D98 115.7 mm to (116.7, 192.9)
- moved MX2 115.7 mm to (126.2, 169.1)
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Connections:
- net Net-(MX10-COL) renamed COL2
- net Net-(MX12-COL) renamed COL3
- net Net-(MX18-COL) renamed COL4
- net Net-(MX24-COL) renamed COL5
- net Net-(MX29-COL) renamed COL6
- net Net-(MX34-COL) renamed COL7
- net Net-(MX40-COL) renamed COL8
- net Net-(MX45-COL) renamed COL9
- net Net-(MX50-COL) renamed COL10
- net Net-(MX56-COL) renamed COL11
- net Net-(MX62-COL) renamed COL12
- net Net-(MX68-COL) renamed COL13
- net Net-(MX73-COL) renamed COL14
- net Net-(MX78-COL) renamed COL15
- net Net-(MX81-COL) renamed COL16
- net Net-(MX85-COL) renamed COL17
- net Net-(MX91-COL) renamed COL18
Other:
- board outline added: 401 x 126 mm

Commit message: added support for 7u and stepped caps
Parts:
- added C1: 1u, Capacitor_SMD:C_0402_1005Metric, F.Cu at (-26.9, 83.3)
- added C10: 22p, Capacitor_SMD:C_0402_1005Metric, F.Cu at (-24.0, 87.2)
- added C11: 22p, Capacitor_SMD:C_0402_1005Metric, F.Cu at (-24.0, 89.2)
- added C12: 1uF, Capacitor_SMD:C_0402_1005Metric, F.Cu at (-24.0, 91.2)
- added C2: 1u, Capacitor_SMD:C_0402_1005Metric, F.Cu at (-26.9, 85.3)
- added C3: 1uF, Capacitor_SMD:C_0402_1005Metric, F.Cu at (-26.9, 87.2)
- added C4: 1uF, Capacitor_SMD:C_0402_1005Metric, F.Cu at (-26.9, 89.2)
- added C5: 10uF, Capacitor_SMD:C_0603_1608Metric, F.Cu at (-23.0, 79.9)
- added C6: 0.1uF, Capacitor_SMD:C_0402_1005Metric, F.Cu at (-26.9, 91.2)
- added C7: 0.1uF, Capacitor_SMD:C_0402_1005Metric, F.Cu at (-26.9, 93.1)
- added C8: 0.1uF, Capacitor_SMD:C_0402_1005Metric, F.Cu at (-24.0, 83.3)
- added C9: 0.1uF, Capacitor_SMD:C_0402_1005Metric, F.Cu at (-24.0, 85.3)
- added D101: SOD-123, Diode_SMD:D_SOD-123, F.Cu at (-25.5, 247.8)
- added D102: SOD-123, Diode_SMD:D_SOD-123, F.Cu at (-25.5, 251.2)
- added D103: SOD-123, Diode_SMD:D_SOD-123, F.Cu at (-25.5, 254.5)
- added D104: SOD-123, Diode_SMD:D_SOD-123, F.Cu at (-25.5, 257.9)
- added D105: SOD-123, Diode_SMD:D_SOD-123, F.Cu at (-25.5, 261.2)
- added D72: SOD-123, Diode_SMD:D_SOD-123, F.Cu at (-37.1, 251.2)
- added D89: SOD-123, Diode_SMD:D_SOD-123, F.Cu at (-31.3, 257.9)
- added F1: Fuse_Small, Fuse:Fuse_1206_3216Metric, F.Cu at (-27.8, 80.2)
- added J1: USB_C_Receptacle_USB2.0_14P, Connector_USB:USB_C_Receptacle_HRO_TYPE-C-31-M-12, F.Cu at (-36.4, 77.6)
- added J2: Conn_01x04, Connector_JST:JST_SH_SM04B-SRSS-TB_1x04-1MP_P1.00mm_Horizontal, F.Cu at (-33.2, 95.4)
- added J3: Conn_01x05, Connector_PinHeader_2.54mm:PinHeader_1x05_P2.54mm_Vertical, F.Cu at (-40.0, 84.6)
- added MX101: MX-NoLED, MX_Only:MXOnly-1.5U-NoLED, B.Cu at (161.9, 219.1)
- added MX102: MX-NoLED, MX_Only:MXOnly-1.5U-NoLED, B.Cu at (323.9, 219.1)
- added MX103: MX-NoLED, MX_Only:MXOnly-1U-NoLED, B.Cu at (347.7, 219.1)
- added MX104: MX-NoLED, MX_Only:MXOnly-1.5U-NoLED, B.Cu at (371.5, 219.1)
- added MX105: MX-NoLED, MX_Only:MXOnly-7U-NoLED, B.Cu at (242.9, 219.1)
- added MX72: MX-NoLED, MX_Only:MXOnly-1.75U-NoLED, F.Cu at (126.2, 181.0)
- added MX89: MX-NoLED, MX_Only:MXOnly-1U-NoLED, B.Cu at (138.1, 219.1)
- added R1: 5.1k, Resistor_SMD:R_0402_1005Metric, F.Cu at (-21.1, 92.2)
- added R2: 5.1k, Resistor_SMD:R_0402_1005Metric, F.Cu at (-21.1, 94.2)
- added R3: 27, Resistor_SMD:R_0402_1005Metric, F.Cu at (-21.1, 96.2)
- added R4: 27, Resistor_SMD:R_0402_1005Metric, F.Cu at (-18.2, 92.2)
- added R5: 1K, Resistor_SMD:R_0402_1005Metric, F.Cu at (-18.2, 94.2)
- added R6: 5.1k, Resistor_SMD:R_0402_1005Metric, F.Cu at (-18.2, 96.2)
- added R7: 1K, Resistor_SMD:R_0402_1005Metric, F.Cu at (-15.3, 92.2)
- added R8: 5.1k, Resistor_SMD:R_0402_1005Metric, F.Cu at (-15.3, 94.2)
- added R9: 5.1k, Resistor_SMD:R_0402_1005Metric, F.Cu at (-15.3, 96.2)
- added SW1: SW_Push, Button_Switch_SMD:SW_Push_SPST_NO_Alps_SKRK, F.Cu at (-19.3, 84.5)
- added SW2: SW_Push, Button_Switch_SMD:SW_Push_SPST_NO_Alps_SKRK, F.Cu at (-19.3, 89.0)
- added U1: RP2040, Package_DFN_QFN:QFN-56-1EP_7x7mm_P0.4mm_EP3.2x3.2mm, F.Cu at (-33.0, 87.0)
- added U2: XC6206PxxxMR, Package_TO_SOT_SMD:SOT-23-3, F.Cu at (-17.7, 74.2)
- added U3: SRV05-4, Package_TO_SOT_SMD:SOT-23-6, F.Cu at (-17.7, 78.9)
- added U4: W25Q128JVS, Package_SO:SOIC-8_5.23x5.23mm_P1.27mm, F.Cu at (-25.4, 75.2)
- added Y1: Crystal_GND24, Crystal:Crystal_SMD_3225-4Pin_3.2x2.5mm, F.Cu at (-25.7, 96.3)
- D1, D10, D100, D11, D12, D13, D14, D15, D16, D17, D18, D19, D2, D20, D21, D22, D23, D24, D25, D26, D27, D28, D29, D3, D30, D31, D32, D33, D34, D35, D36, D37, D38, D39, D4, D40, D41, D42, D43, D44, D45, D46, D47, D48, D49, D5, D50, D51, D52, D53, D54, D55, D56, D57, D58, D59, D6, D60, D61, D62, D63, D64, D65, D66, D67, D68, D69, D7, D70, D71, D73, D74, D75, D76, D77, D78, D79, D8, D80, D81, D82, D83, D84, D85, D86, D87, D88, D9, D90, D91, D92, D93, D94, D95, D96, D97, D98, D99: moved to F.Cu
- MX78: footprint MX_Only:MXOnly-1U-NoLED -> MX_Only:MXOnly-1.5U-NoLED; moved to B.Cu
- MX9: footprint MX_Only:MXOnly-1.75U-NoLED -> MX_Only:MXOnly-1.75U
- moved D91 520.5 mm to (-25.5, 214.3), turned to 0 degrees
- moved D92 517.5 mm to (-25.5, 217.7), turned to 0 degrees
- moved D93 515.8 mm to (-25.5, 221.0), turned to 0 degrees
- moved D94 513.7 mm to (-25.5, 224.4), turned to 0 degrees
- moved D85 513.1 mm to (-31.3, 244.5), turned to 0 degrees
- moved D86 508.9 mm to (-31.3, 247.8), turned to 0 degrees
- moved D87 506.3 mm to (-31.3, 251.2), turned to 0 degrees
- moved D88 502.2 mm to (-31.3, 254.5), turned to 0 degrees
- moved D90 501.3 mm to (-31.3, 261.2), turned to 0 degrees
- moved D81 491.6 mm to (-31.3, 231.1), turned to 0 degrees
- moved D82 487.9 mm to (-31.3, 234.4), turned to 0 degrees
- moved D83 485.5 mm to (-31.3, 237.8), turned to 0 degrees
- moved D84 481.4 mm to (-31.3, 241.1), turned to 0 degrees
- moved D78 466.3 mm to (-31.3, 221.0), turned to 0 degrees
- moved D73 463.9 mm to (-37.1, 254.5), turned to 0 degrees
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Connections:
- D78 pad 1: ROW0 -> ROW5
- MX73 pad 1: COL14 -> COL15
- MX77 pad 1: COL14 -> COL15
- MX78 pad 1: COL15 -> COL2
Other:
- board size 401 x 126 mm -> 419.1 x 157.2 mm

Commit message: placed diodes
Parts:
- D1, D10, D100, D101, D102, D103, D104, D105, D11, D12, D13, D14, D15, D16, D17, D18, D19, D2, D20, D21, D22, D23, D24, D25, D26, D27, D28, D29, D3, D30, D31, D32, D33, D34, D35, D36, D37, D38, D39, D4, D40, D41, D42, D43, D44, D45, D46, D47, D48, D49, D5, D50, D51, D52, D53, D54, D55, D56, D57, D58, D59, D6, D60, D61, D62, D63, D64, D65, D66, D67, D68, D69, D7, D70, D71, D72, D73, D74, D75, D76, D77, D78, D79, D8, D80, D81, D82, D83, D84, D85, D86, D87, D88, D89, D9, D90, D91, D92, D93, D94, D95, D96, D97, D98, D99: moved to B.Cu
- moved D34 308.4 mm to (242.9, 123.8), turned to 90 degrees
- moved D29 300.3 mm to (214.3, 123.8), turned to 90 degrees
- moved D38 288.7 mm to (238.1, 204.8), turned to 90 degrees
- moved D37 281.5 mm to (228.6, 185.7), turned to 90 degrees
- moved D36 280.0 mm to (223.8, 166.7), turned to 90 degrees
- moved D24 275.9 mm to (195.3, 123.8), turned to 90 degrees
- moved D35 274.9 mm to (214.3, 147.6), turned to 90 degrees
- moved D30 274.5 mm to (195.5, 147.6), turned to 90 degrees
- moved D33 268.2 mm to (219.1, 204.8), turned to 90 degrees
- moved D32 260.2 mm to (209.6, 185.7), turned to 90 degrees
- moved D28 259.3 mm to (200.0, 204.8), turned to 90 degrees
- moved D31 257.9 mm to (204.8, 166.7), turned to 90 degrees
- moved D26 253.7 mm to (185.9, 166.6), turned to 90 degrees
- moved D27 253.5 mm to (190.5, 185.7), turned to 90 degrees
- moved D12 251.9 mm to (157.2, 123.8), turned to 90 degrees
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
Commit message: finished diode layout
Parts:
- removed C1, C2: 1u, Capacitor_SMD:C_0402_1005Metric
- removed C10, C11: 22p, Capacitor_SMD:C_0402_1005Metric
- removed C12, C3, C4: 1uF, Capacitor_SMD:C_0402_1005Metric
- removed C5: 10uF, Capacitor_SMD:C_0603_1608Metric
- removed C6, C7, C8, C9: 0.1uF, Capacitor_SMD:C_0402_1005Metric
- removed F1: Fuse_Small, Fuse:Fuse_1206_3216Metric
- removed J1: USB_C_Receptacle_USB2.0_14P, Connector_USB:USB_C_Receptacle_HRO_TYPE-C-31-M-12
- removed J2: Conn_01x04, Connector_JST:JST_SH_SM04B-SRSS-TB_1x04-1MP_P1.00mm_Horizontal
- removed J3: Conn_01x05, Connector_PinHeader_2.54mm:PinHeader_1x05_P2.54mm_Vertical
- removed R1, R2, R6, R8, R9: 5.1k, Resistor_SMD:R_0402_1005Metric
- removed R3, R4: 27, Resistor_SMD:R_0402_1005Metric
- removed R5, R7: 1K, Resistor_SMD:R_0402_1005Metric
- removed SW1, SW2: SW_Push, Button_Switch_SMD:SW_Push_SPST_NO_Alps_SKRK
- removed U1: RP2040, Package_DFN_QFN:QFN-56-1EP_7x7mm_P0.4mm_EP3.2x3.2mm
- removed U2: XC6206PxxxMR, Package_TO_SOT_SMD:SOT-23-3
- removed U3: SRV05-4, Package_TO_SOT_SMD:SOT-23-6
- removed U4: W25Q128JVS, Package_SO:SOIC-8_5.23x5.23mm_P1.27mm
- removed Y1: Crystal_GND24, Crystal:Crystal_SMD_3225-4Pin_3.2x2.5mm
- moved D90 494.7 mm to (428.6, 223.8)
- moved D85 488.8 mm to (428.6, 123.8)
- moved D88 488.4 mm to (428.6, 204.8)
- moved D87 488.3 mm to (428.6, 166.7)
- moved D86 487.7 mm to (428.6, 147.6)
- moved D94 476.9 mm to (447.7, 223.8)
- moved D91 476.7 mm to (447.7, 123.8)
- moved D93 476.6 mm to (447.7, 166.7)
- moved D92 475.8 mm to (447.7, 147.6)
- moved D74 461.3 mm to (385.8, 123.8)
- moved D81 457.1 mm to (409.6, 123.8)
- moved D83 456.1 mm to (409.6, 166.7)
- moved D82 455.7 mm to (409.6, 147.6)
- moved D84 455.5 mm to (409.6, 223.8)
- moved D104 448.5 mm to (385.8, 219.1)
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
Commit message: flipped keys for tsangan layout to be on correct plane
Parts:
- MX101, MX102, MX103, MX104, MX105, MX78, MX89: moved to F.Cu
- MX9: footprint MX_Only:MXOnly-1.75U -> MX_Only:MXOnly-1.75U-NoLED
- moved D104 8.33 mm to (385.8, 227.4), turned to -90 degrees
- moved D78 3.67 mm to (123.8, 227.5), turned to -90 degrees
- moved D101 3.61 mm to (171.4, 227.4)
- moved D102 3.61 mm to (338.1, 227.4)
- moved D103 3.61 mm to (357.2, 227.4)
- moved D89 3.61 mm to (147.6, 227.4)
- moved D11 2.44 mm to (123.8, 221.5)
- moved D17 2.42 mm to (147.6, 221.5), turned to 90 degrees
- moved D23 2.42 mm to (171.4, 221.5), turned to 90 degrees
- moved D61 2.42 mm to (338.1, 221.5), turned to 90 degrees
- moved D67 2.42 mm to (357.2, 221.5), turned to 90 degrees
- moved D73 2.38 mm to (385.8, 221.5)
- turned MX101 to 180 degrees
- turned MX102 to 180 degrees
- turned MX103 to 180 degrees
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Other:
- board size 419.1 x 157.2 mm -> 400.1 x 128.6 mm

Commit message: rotated keys for tsangan layout and stepped caps to be proper orientation.
Parts:
- added C1: 1u, Capacitor_SMD:C_0402_1005Metric, F.Cu at (-25.2, 112.1)
- added C2: 1u, Capacitor_SMD:C_0402_1005Metric, F.Cu at (-25.2, 114.1)
- added F1: Fuse_Small, Fuse:Fuse_1206_3216Metric, F.Cu at (-26.1, 109.1)
- added J1: USB_C_Receptacle_USB2.0_14P, Connector_USB:USB_C_Receptacle_HRO_TYPE-C-31-M-12, F.Cu at (-34.7, 106.5)
- added J2: Conn_01x04, Connector_JST:JST_SH_SM04B-SRSS-TB_1x04-1MP_P1.00mm_Horizontal, F.Cu at (-31.5, 124.3)
- added R1: 5.1k, Resistor_SMD:R_0402_1005Metric, F.Cu at (-19.4, 121.0)
- added R2: 5.1k, Resistor_SMD:R_0402_1005Metric, F.Cu at (-19.4, 123.0)
- added R6: 5.1k, Resistor_SMD:R_0402_1005Metric, F.Cu at (-16.5, 125.0)
- added R7: 1K, Resistor_SMD:R_0402_1005Metric, F.Cu at (-13.6, 121.0)
- added R8: 5.1k, Resistor_SMD:R_0402_1005Metric, F.Cu at (-13.6, 123.0)
- added R9: 5.1k, Resistor_SMD:R_0402_1005Metric, F.Cu at (-13.6, 125.0)
- added SW1: SW_Push, Button_Switch_SMD:SW_Push_SPST_NO_Alps_SKRK, F.Cu at (-17.6, 113.4)
- added SW2: SW_Push, Button_Switch_SMD:SW_Push_SPST_NO_Alps_SKRK, F.Cu at (-17.6, 117.8)
- added U1: ESP32-S2, Package_DFN_QFN:QFN-56-1EP_7x7mm_P0.4mm_EP5.6x5.6mm, F.Cu at (-31.3, 115.8)
- added U2: XC6206PxxxMR, Package_TO_SOT_SMD:SOT-23-3, F.Cu at (-16.0, 103.1)
- added U3: SRV05-4, Package_TO_SOT_SMD:SOT-23-6, F.Cu at (-16.0, 107.7)
- moved MX72 4.76 mm to (121.4, 181.0)
- turned MX101 to 0 degrees
- turned MX102 to 0 degrees
- turned MX103 to 0 degrees
- turned MX104 to 0 degrees
- turned MX105 to 0 degrees
- turned MX78 to 0 degrees
- turned MX89 to 0 degrees
Connections:
- MX102 pad 1: COL10 -> COL11
- MX103 pad 1: COL11 -> COL13
- MX104 pad 1: COL12 -> COL15
- MX34 pad 1: COL7 -> COL8
- MX40 pad 1: COL8 -> COL9
- MX45 pad 1: COL9 -> COL10
- MX50 pad 1: COL10 -> COL11
- MX56 pad 1: COL11 -> COL12
- MX62 pad 1: COL12 -> COL13
- MX67 pad 1: COL12 -> COL13
- MX68 pad 1: COL13 -> COL14
- MX74 pad 1: COL14 -> COL15

Commit message: added support for f13 row
Parts:
- added D106: SOD-123, Diode_SMD:D_SOD-123, F.Cu at (69.6, 58.2)
- added D107: SOD-123, Diode_SMD:D_SOD-123, F.Cu at (69.6, 61.5)
- added D108: SOD-123, Diode_SMD:D_SOD-123, F.Cu at (69.6, 64.9)
- added D109: SOD-123, Diode_SMD:D_SOD-123, F.Cu at (69.6, 68.2)
- added D110: SOD-123, Diode_SMD:D_SOD-123, F.Cu at (69.6, 71.6)
- added D111: SOD-123, Diode_SMD:D_SOD-123, F.Cu at (75.4, 58.2)
- added D112: SOD-123, Diode_SMD:D_SOD-123, F.Cu at (75.4, 61.5)
- added D113: SOD-123, Diode_SMD:D_SOD-123, F.Cu at (75.4, 64.9)
- added D114: SOD-123, Diode_SMD:D_SOD-123, F.Cu at (75.4, 68.2)
- added MX106: MX-NoLED, MX_Only:MXOnly-1U-NoLED, F.Cu at (133.3, 119.1)
- added MX107: MX-NoLED, MX_Only:MXOnly-1U-NoLED, F.Cu at (152.4, 119.1)
- added MX108: MX-NoLED, MX_Only:MXOnly-1U-NoLED, F.Cu at (171.4, 119.1)
- added MX109: MX-NoLED, MX_Only:MXOnly-1U-NoLED, F.Cu at (190.5, 119.1)
- added MX110: MX-NoLED, MX_Only:MXOnly-1U-NoLED, F.Cu at (214.3, 119.1)
- added MX111: MX-NoLED, MX_Only:MXOnly-1U-NoLED, F.Cu at (295.3, 119.1)
- added MX112: MX-NoLED, MX_Only:MXOnly-1U-NoLED, F.Cu at (314.3, 119.1)
- added MX113: MX-NoLED, MX_Only:MXOnly-1U-NoLED, F.Cu at (333.4, 119.1)
- added MX114: MX-NoLED, MX_Only:MXOnly-1U-NoLED, F.Cu at (352.4, 119.1)
