File: tklx/tklx.kicad_sch (KiCad schematic)
At the start: 240 parts, among them J1 USB_C_Receptacle_USB2.0_14P, SW1 SW_Push, U1 TLV75801PDRV, U2 XC6206PxxxMR, U3 SRV05-4, U4 ESP32-S3

Commit message: finished esp32 wireless design
Parts:
- removed F1: Fuse_Small, Fuse:Fuse_1206_3216Metric, symbol Device:Fuse_Small
- removed U1: TLV75801PDRV, Package_SON:WSON-6-1EP_2x2mm_P0.65mm_EP1x1.6mm, symbol Regulator_Linear:TLV75801PDRV
- removed U2: XC6206PxxxMR, Package_TO_SOT_SMD:SOT-23-3, symbol Regulator_Linear:XC6206PxxxMR
- removed U3: SRV05-4, Package_TO_SOT_SMD:SOT-23-6, symbol Power_Protection:SRV05-4
- added ANT1: 2450AT18D0100E, Samacsys:2450AT18D0100E, symbol Samacsys:2450AT18D0100E
- added C10, C13, C4, C8: 1uF, Capacitor_SMD:C_0805_2012Metric, symbol Device:C_Small
- added C11, C12, C14, C5, C6, C9: 0.1uF, Capacitor_SMD:C_0805_2012Metric, symbol Device:C_Small
- added C15, C16: 12pF, Capacitor_SMD:C_0805_2012Metric, symbol Device:C_Small
- added C17, C18: NC, Capacitor_SMD:C_0805_2012Metric, symbol Device:C_Small
- added C19: 2.4pF, Capacitor_SMD:C_0805_2012Metric, symbol Device:C_Small
- added C20: 2.7pF, Capacitor_SMD:C_0805_2012Metric, symbol Device:C_Small
- added C3: 10uF, Capacitor_SMD:C_0805_2012Metric, symbol Device:C_Small
- added C7: 10nF, Capacitor_SMD:C_0805_2012Metric, symbol Device:C_Small
- added D115: PMEG6020AELR, symbol Device:D_Schottky
- added D116: PTVS5V0Z1USKP, Diode_SMD:Nexperia_DSN1608-2_1.6x0.8mm, symbol Diode:PTVS5V0Z1USKP
- added L1: 2nH, symbol Device:L_Small
- added L2: 2.4nH, symbol Device:L
- added R10: 22, Resistor_SMD:R_0402_1005Metric, symbol Device:R_Small
- added R11, R3, R4, R5, R7, R8: 0, Resistor_SMD:R_0402_1005Metric, symbol Device:R_Small
- added R9: 100K, symbol Device:R_Small
- added SW2: SW_SPST, Button_Switch_SMD:SW_Push_SPST_NO_Alps_SKRK, symbol Switch:SW_SPST
- added U1: TLV76733DRVx, Package_SON:WSON-6-1EP_2x2mm_P0.65mm_EP1x1.6mm_ThermalVias, symbol Regulator_Linear:TLV76733DRVx
- added U2: USBLC6-2P6, Package_TO_SOT_SMD:SOT-666, symbol Power_Protection:USBLC6-2P6
- added U5: W25Q128JVP, Package_SON:WSON-8-1EP_6x5mm_P1.27mm_EP3.4x4.3mm, symbol Memory_Flash:W25Q128JVP
- added Y1: ECS-400-10-37B2-CKM-TR, symbol Device:Crystal_GND24_Small
- C1: value 1u -> 1uF; footprint Capacitor_SMD:C_0402_1005Metric -> Capacitor_SMD:C_0805_2012Metric
- C2: value 1u -> 2.2uF; footprint Capacitor_SMD:C_0402_1005Metric -> Capacitor_SMD:C_0805_2012Metric
- R6: value 5.1k -> 10k
Connections:
- net +3V3: now also U4.20 (VDD3P3_RTC), U4.46 (VDD3P3_CPU), U4.55 (VDDA), U4.56 (VDDA), C12.1, C3.1, C4.1, C5.1, C7.1, C8.1, C9.1, L1.1, U1.1 (OUT), U1.2 (SNS)
- net BOOT: now also SW2.1 (A)
- net D+: now also U2.4 (I/O2)
- net D-: now also U2.6 (I/O1)
- net GND: now also ANT1.2 (GND_1), ANT1.3 (GND_2), ANT1.4 (GND/FEED), C10.2, C11.2, C12.2, C13.2, C14.2, C15.2, C16.2, C17.1, C18.1, C19.1, C20.1, C3.2, C4.2, C5.2, C6.2, C7.2, C8.2, C9.2, D116.2 (A), SW2.2 (B), U1.3 (GND), U1.5 (GND), U1.7 (PAD), U2.2 (GND), U5.4 (GND), Y1.2, Y1.4; no longer J1.S1 (SHIELD)
- net RESET: now also C13.1
- net VBUS: now also C14.1, D115.1 (K), U2.5 (VBUS)
- net VDD3P3: now also C6.1, L1.2
- net LNA_IN: now reaches U4.1 (LNA_IN/RF)
- net LNA_IN: now also C20.2, L2.2
- net SPICS1: now reaches U4.28 (SPI_CS1/GPIO26)
- net VDD_SPI: now reaches U4.29 (VDD_SPI)
- net VDD_SPI: now also C10.1, C11.1
- net at U4.30 (SPIHD/GPIO27): now also R3.2
- net at U4.31 (SPIWP/GPIO28): now also R4.2
- net SPICS0: now reaches U4.32 (SPICS0/GPIO29)
- net SPICS0: now also R9.2, U5.1 (~{CS})
- net at U4.33 (SPICLK/GPIO30): now also R5.2
- net at U4.34 (SPIQ/GPIO31): now also R7.2
- net at U4.35 (SPID/GPIO32): now also R8.1
- net XTAL_N: now reaches U4.53 (XTAL_N)
- net XTAL_P: now reaches U4.54 (XTAL_P)
- net +5V renamed VIN
- net VIN: now also D115.2 (A), D116.1 (K), U1.4 (EN), U1.6 (IN)
- new net: C18.2, C19.2, L2.1, R11.2
- new net: ANT1.1 (FEED/GND), C17.2, R11.1
- new net: R9.1, U5.8 (VCC)
- new net: C15.1, R10.2, Y1.1
- new net D_N: U2.1 (I/O1)
- new net D_P: U2.3 (I/O2)
- new net SPICLK: R5.1, U5.6 (CLK)
- new net SPID: R8.2, U5.5 (DI(IO0))
- new net SPIHD: R3.1, U5.7 (IO3)
- new net SPIQ: R7.1, U5.2 (DO(IO1))
- new net SPIWP: R4.1, U5.3 (IO2)
- new net XATL_N: C16.1, Y1.3
- new net XATL_P: R10.1
- no-connect marks 6 -> 11
Other:
- moved on the sheet: R6, SW1, U4

Commit message: prelim esp32-mini design
Parts:
- removed ANT1: 2450AT18D0100E, Samacsys:2450AT18D0100E, symbol Samacsys:2450AT18D0100E
- removed C10, C13, C8: 1uF, Capacitor_SMD:C_0805_2012Metric, symbol Device:C_Small
- removed C11, C12, C14, C9: 0.1uF, Capacitor_SMD:C_0805_2012Metric, symbol Device:C_Small
- removed C15, C16: 12pF, Capacitor_SMD:C_0805_2012Metric, symbol Device:C_Small
- removed C17, C18: NC, Capacitor_SMD:C_0805_2012Metric, symbol Device:C_Small
- removed C19: 2.4pF, Capacitor_SMD:C_0805_2012Metric, symbol Device:C_Small
- removed C20: 2.7pF, Capacitor_SMD:C_0805_2012Metric, symbol Device:C_Small
- removed C7: 10nF, Capacitor_SMD:C_0805_2012Metric, symbol Device:C_Small
- removed D115: PMEG6020AELR, symbol Device:D_Schottky
- removed D116: PTVS5V0Z1USKP, Diode_SMD:Nexperia_DSN1608-2_1.6x0.8mm, symbol Diode:PTVS5V0Z1USKP
- removed J1: USB_C_Receptacle_USB2.0_14P, Connector_USB:USB_C_Receptacle_HRO_TYPE-C-31-M-12, symbol Connector:USB_C_Receptacle_USB2.0_14P
- removed L1: 2nH, symbol Device:L_Small
- removed L2: 2.4nH, symbol Device:L
- removed R10: 22, Resistor_SMD:R_0402_1005Metric, symbol Device:R_Small
- removed R11, R3, R4, R5, R7, R8: 0, Resistor_SMD:R_0402_1005Metric, symbol Device:R_Small
- removed R6: 10k, Resistor_SMD:R_0402_1005Metric, symbol Device:R_Small
- removed R9: 100K, symbol Device:R_Small
- removed SW2: SW_SPST, Button_Switch_SMD:SW_Push_SPST_NO_Alps_SKRK, symbol Switch:SW_SPST
- removed U1: TLV76733DRVx, Package_SON:WSON-6-1EP_2x2mm_P0.65mm_EP1x1.6mm_ThermalVias, symbol Regulator_Linear:TLV76733DRVx
- removed U2: USBLC6-2P6, Package_TO_SOT_SMD:SOT-666, symbol Power_Protection:USBLC6-2P6
- removed U4: ESP32-S3, Package_DFN_QFN:QFN-56-1EP_7x7mm_P0.4mm_EP5.6x5.6mm, symbol PCM_Espressif:ESP32-S3
- removed U5: W25Q128JVP, Package_SON:WSON-8-1EP_6x5mm_P1.27mm_EP3.4x4.3mm, symbol Memory_Flash:W25Q128JVP
- removed Y1: ECS-400-10-37B2-CKM-TR, symbol Device:Crystal_GND24_Small
- added J1: Conn_01x04, Connector_JST:JST_EH_S4B-EH_1x04_P2.50mm_Horizontal, symbol Connector_Generic:Conn_01x04
- added SW2: SW_Push, Button_Switch_SMD:SW_Push_1P1T_XKB_TS-1187A, symbol Switch:SW_Push
- added U1: AMS1117-3.3, Package_TO_SOT_SMD:SOT-223-3_TabPin2, symbol Regulator_Linear:AMS1117-3.3
- added U3: ESP32-S3-MINI-1, RF_Module:ESP32-S2-MINI-1, symbol RF_Module:ESP32-S3-MINI-1
- C1: value 1uF -> 10uF
- C2: value 2.2uF -> 10uF
- C3: value 10uF -> 100nF
- C4: value 1uF -> 22uF
- C5: value 0.1uF -> 1uF
- C6: value 0.1uF -> 100nF
- R1: value 5.1k -> 10k; footprint Resistor_SMD:R_0402_1005Metric -> Resistor_SMD:R_0805_2012Metric
- R2: value 5.1k -> 100; footprint Resistor_SMD:R_0402_1005Metric -> Resistor_SMD:R_0805_2012Metric
- SW1: footprint Button_Switch_SMD:SW_Push_SPST_NO_Alps_SKRK -> Button_Switch_SMD:SW_Push_1P1T_XKB_TS-1187A
Connections:
- net RESET is gone; now on net GND: SW1.2
- net VDD3P3 is gone; now on net GND: C6.1
- net VIN is gone; now on net +3.3V: C1.1
- net BOOT: now also R2.1, U3.4 (IO0)
- net COL0: now also U3.5 (IO1)
- net COL1: now also U3.6 (IO2)
- net COL10: now also U3.15 (IO11)
- net COL11: now also U3.16 (IO12)
- net COL12: now also U3.17 (IO13)
- net COL13: now also U3.18 (IO14)
- net COL14: now also U3.19 (IO15)
- net COL15: now also U3.20 (IO16)
- net COL16: now also U3.21 (IO17)
- net COL17: now also U3.22 (IO18)
- net COL18: now also U3.25 (IO21)
- net COL2: now also U3.7 (IO3)
- net COL3: now also U3.8 (IO4)
- net COL4: now also U3.9 (IO5)
- net COL5: now also U3.10 (IO6)
- net COL6: now also U3.11 (IO7)
- net COL7: now also U3.12 (IO8)
- net COL8: now also U3.13 (IO9)
- net COL9: now also U3.14 (IO10)
- net D+: now also J1.2 (Pin_2), U3.24 (USB_D+)
- net D-: now also J1.3 (Pin_3), U3.23 (USB_D-)
- net GND: now also J1.4 (Pin_4), SW2.2, U1.1 (GND), U3.1 (GND), U3.2 (GND), U3.42 (GND), U3.43 (GND), U3.46 (GND), U3.47 (GND), U3.48 (GND), U3.49 (GND), U3.50 (GND), U3.51 (GND), U3.52 (GND), U3.53 (GND), U3.54 (GND), U3.55 (GND), U3.56 (GND), U3.57 (GND), U3.58 (GND), U3.59 (GND), U3.60 (GND), U3.61 (GND), U3.62 (GND), U3.63 (GND), U3.64 (GND), U3.65 (GND); no longer C6.2, R1.2, R2.2, SW1.1
- net ROW0: now also U3.26 (IO26)
- net ROW1: now also U3.28 (IO33)
- net ROW2: now also U3.29 (IO34)
- net ROW3: now also U3.31 (IO35)
- net ROW4: now also U3.32 (IO36)
- net ROW5: now also U3.33 (IO37)
- net VBUS: now also J1.1 (Pin_1)
- net +3.3V: now reaches R1.1
- net +3.3V: now also C3.1, C4.1, C6.2, SW1.1, U1.2 (VO), U3.3 (3V3), U3.45 (EN)
- removed net +3V3: C2.1, C3.1, C4.1, C5.1
- new net: C5.1, R1.2
- new net: R2.2, SW2.1
- new net +5V: C2.1, U1.3 (VI)
